File: esp_extension/esp_extension.kicad_sch (KiCad schematic)
At the start: 66 parts, among them J1 MOTOR1, J10 MPU6050, J2 MOTOR2, J3 MOTOR3, J4 MOTOR4, J5 ESP32-S3-LeftHeader, J6 BATTERY, J7 ESP32-S3-RightHeader, J8 I2C, J9 GPIO, Q1 AO3400A, Q2 AO3400A, Q3 AO3400A, Q4 AO3400A, SW1 SW_SPDT, U2 TPS63802DLAR, U3 MS5611-01BA

Commit message: JLC production files
Parts:
- D5: Manufacturer R+O -> Hongjiacheng
Changed lines of the file:
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@@
 			)
 		)
-		(property "Manufacturer" "R+O"
+		(property "Manufacturer" "Hongjiacheng"
 			(at 82.55 187.96 90)
 			(hide yes)
